Commit message: change linear axis values

File: setup/catkin/princeton_cell/urdf/full_cell.urdf (robot description, URDF)
Before this commit: robot full_cell, 23 links, 22 joints
Joints:
- joint A_cart_joint: limit lower=-1.926 upper=0.675 effort=100000 velocity=2.618 -> lower=0.0 upper=4.0 effort=100000 velocity=2.618
- joint B_cart_joint: limit lower=-1.926 upper=0.675 effort=100000 velocity=2.618 -> lower=0.0 upper=4.0 effort=100000 velocity=2.618

File: setup/catkin/princeton_cell/urdf/full_cell_macro.xacro (robot description, xacro)
@@ -14,5 +14,5 @@
       <parent link="world" />
       <child link = "B_axis" />
-      <origin xyz="0.0 0.0 0.0" rpy="0.0 0.0 0.0" />
+      <origin rpy="0.0 0.0 3.14159" xyz="3.70 3.45 0.02"/>
     </joint>
     <xacro:abb_on_axis prefix="B_"/>

File: setup/catkin/princeton_cell/urdf/linear_axis.xacro (robot description, xacro)
@@ -25,5 +25,5 @@
       <origin xyz="0 0 0" rpy="0 0 0 "/>
       <axis   xyz="1 0 0"/>
-      <limit lower="-1.926" upper="0.675" effort="100000" velocity="2.618" />
+      <limit lower="0" upper="4.0" effort="100000" velocity="2.618" />
       <dynamics damping="0.2" friction="0" />
     </joint>
